Commit message: phuongnho

File: my_robot_description/urdf/macros2.xacro (robot description, xacro)
@@ -11,5 +11,5 @@
               <origin rpy="0 1.5707 1.5707" xyz="0 0 0"/>
               <geometry>
-                <cylinder length="0.05" radius="0.09"/>
+                <cylinder length="0.05" radius="0.0275"/>
               </geometry>
             </collision>
@@ -17,5 +17,5 @@
               <origin rpy="0 1.5707 1.5707" xyz="0 0 0"/>
               <geometry>
-                <cylinder length="0.05" radius="0.09"/>
+                <cylinder length="0.05" radius="0.0275"/>
               </geometry>
             </visual>

File: my_robot_description/urdf/my_robot2.urdf.xacro (robot description, xacro)
@@ -21,5 +21,5 @@
         <collision name="collision_base_link">
             <geometry>
-                <box size="0.55 0.3 0.15"/>
+                <box size="0.55 0.3 0.11"/>
             </geometry>
         </collision>
@@ -32,4 +32,9 @@
         </visual>
     </link>
+    <joint name="scan_joint" type="fixed">
+        <origin xyz="-0.045 0 0.08" rpy="0 0 0"/>
+        <parent link="base_link"/>
+        <child link="base_scan"/>
+    </joint>
     <link name="base_scan">
         <inertial>
@@ -52,20 +57,36 @@
         </collision>
     </link>
-    <joint name="scan_joint" type="fixed">
-        <origin xyz="-0.045 0 0.08" rpy="0 0 0"/>
+    <joint name="caster_back_joint" type="fixed">
         <parent link="base_link"/>
-        <child link="base_scan"/>
+        <child link="caster_back_link"/>
+        <origin xyz=" 0 0 0" rpy="0 0 0"/>
     </joint>
-    <xacro:link_wheel name="blink_right_wheel" />
-    <xacro:joint_wheel name="bjoint_right_wheel" child="blink_right_wheel" origin_xyz="-0.18 0.17 -0.06" />
-    <xacro:link_wheel name="blink_left_wheel" />
-    <xacro:joint_wheel name="bjoint_left_wheel" child="blink_left_wheel" origin_xyz="-0.18 -0.17 -0.06" />
-    <xacro:link_wheel name="mlink_right_wheel" />
-    <xacro:joint_wheel name="mjoint_right_wheel" child="mlink_right_wheel" origin_xyz="0.0 0.17 -0.06" />
-    <xacro:link_wheel name="mlink_left_wheel" />
-    <xacro:joint_wheel name="mjoint_left_wheel" child="mlink_left_wheel" origin_xyz="0.0 -0.17 -0.06" />
-    <xacro:link_wheel name="flink_right_wheel" />
-    <xacro:joint_wheel name="fjoint_right_wheel" child="flink_right_wheel" origin_xyz="0.18 0.17 -0.06" />
-    <xacro:link_wheel name="flink_left_wheel" />
-    <xacro:joint_wheel name="fjoint_left_wheel" child="flink_left_wheel" origin_xyz="0.18 -0.17 -0.06" />
+    <link name="caster_back_link">
+        <collision>
+            <origin rpy=" 0 0 0" xyz="0.4 0 -0.0374"/>
+            <geometry>
+                <sphere radius="0.05"/>
+            </geometry>
+            <surface>
+                <friction>
+                <ode>
+                    <mu>0</mu>
+                    <mu2>0</mu2>
+                    <slip1>1.0</slip1>
+                    <slip2>1.0</slip2>
+                </ode>
+                </friction>
+            </surface>
+        </collision>
+        <visual>
+            <origin rpy=" 0 0 0" xyz="0.2 0 -0.0374"/>
+            <geometry>
+                <sphere radius="0.05"/>
+            </geometry>
+        </visual>
+    </link>
+    <xacro:link_wheel name="wheel_right_link" />
+    <xacro:joint_wheel name="wheel_right_joint" child="wheel_right_link" origin_xyz="-0.18 0.17 -0.06" />
+    <xacro:link_wheel name="wheel_left_link" />
+    <xacro:joint_wheel name="wheel_left_joint" child="wheel_left_link" origin_xyz="-0.18 -0.17 -0.06" />
 </robot>

Commit message: good

File: my_robot_description/urdf/macros2.xacro (robot description, xacro)
@@ -11,5 +11,5 @@
               <origin rpy="0 1.5707 1.5707" xyz="0 0 0"/>
               <geometry>
-                <cylinder length="0.05" radius="0.0275"/>
+                <cylinder length="0.05" radius="0.022"/>
               </geometry>
             </collision>
@@ -17,5 +17,5 @@
               <origin rpy="0 1.5707 1.5707" xyz="0 0 0"/>
               <geometry>
-                <cylinder length="0.05" radius="0.0275"/>
+                <cylinder length="0.05" radius="0.022"/>
               </geometry>
             </visual>

Commit message: Revert "good"
This reverts commit 42638dec81e677e838e842fa1ea0ccc986494528.

File: my_robot_description/urdf/macros2.xacro (robot description, xacro)
@@ -11,5 +11,5 @@
               <origin rpy="0 1.5707 1.5707" xyz="0 0 0"/>
               <geometry>
-                <cylinder length="0.05" radius="0.022"/>
+                <cylinder length="0.05" radius="0.0275"/>
               </geometry>
             </collision>
@@ -17,5 +17,5 @@
               <origin rpy="0 1.5707 1.5707" xyz="0 0 0"/>
               <geometry>
-                <cylinder length="0.05" radius="0.022"/>
+                <cylinder length="0.05" radius="0.0275"/>
               </geometry>
             </visual>
